Commit message: new

File: src/turn_on_wheeltec_robot/urdf/mini_akm_robot.urdf (robot description, URDF)
Before this commit: robot wheeltec_robot, 5 links, 4 joints
Links:
- removed link base_link
- added link ugv_base_link; visual box size=0.23 0.11 0.05
Joints:
- joint left_front_joint: parent base_link -> ugv_base_link
- joint left_wheel_joint: parent base_link -> ugv_base_link
- joint right_front_joint: parent base_link -> ugv_base_link
- joint right_wheel_joint: parent base_link -> ugv_base_link
